Commit message: new

File: urdf/bjh_model.urdf (robot description, URDF)
Before this commit: robot human_model, 58 links, 57 joints
Links:
- added link fetch_middle
- added link fetch_position
- added link lHand_alter
- added link rHand_alter
- added link rHand_middle
Joints:
- added joint fetch_middle_fetch_position: type fixed, parent fetch_middle, child fetch_position, origin xyz=0.0 0.2 -0.3 rpy=0.0 0.0 2.3561863
- added joint lHand_to_lHand_alter: type fixed, parent lHand, child lHand_alter, origin xyz=0.0 0.0 0.0 rpy=0 -1.5707963 0
- added joint rHand_middle_to_rHand_alter: type fixed, parent rHand_middle, child rHand_alter, origin xyz=0.0 0.0 0.07 rpy=0.0 0.0 0.78539
- added joint rHand_to_rHand_middle: type fixed, parent rHand, child rHand_middle, origin xyz=0.0 0.0 0.0 rpy=0.0 1.5707963 0.0
- added joint spine3_to_fetch_middle: type fixed, parent spine3, child fetch_middle, origin xyz=0.0 0.0 0.0 rpy=-1.5707963 0.0 0.0
